File: docs/electrical/rev_c/Lunar_Hawks_RevC.kicad_sch (KiCad schematic)
At the start: 34 parts, among them J20 CONVEYOR MOTOR, J21 BUCKET ACTUATOR PAIR; SYNC RE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, J22 LIFT ACTUATOR PAIR; SYNC REQU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, K1 DC CONTACTOR - RATING TBD, M1 FL BLDC MOTOR, M2 FR BLDC MOTOR, M3 RL BLDC MOTOR, M4 RR BLDC MOTOR, SW1 LATCHING E-STOP NC, U1 CARRIER INPUT PROTECTION / DC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, U10 FL EXTERNAL BLDC CONTROLLER, U11 FR EXTERNAL BLDC CONTROLLER, U12 RL EXTERNAL BLDC CONTROLLER, U13 RR EXTERNAL BLDC CONTROLLER, U2 JETSON ORIN NX CARRIER - MODE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, U20 CONVEYOR EXTERNAL BRUSHED DRI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, U21 BUCKET EXTERNAL BRUSHED DRIVER, U22 LIFT EXTERNAL BRUSHED DRIVER, U3 ISOLATED UART MODULE 115200, U4 COMPUTE 3V3 REGULATOR MODULE, U5 24V TO 3V3 REGULATOR MODULE, U6 ESP32 WROOM INTERFACE - GPIO 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

Commit message: Correct top-hinged latch door and four-actuator excavation sequence
Parts:
- added F23: LATCH BRANCH FUSE - TBD, symbol Module_F23
- added J23: DOOR / LATCH FEEDBACK INTERFACE, symbol Module_J23
- added J24: ACTUATOR ENDPOINT FEEDBACK, symbol Module_J24
- added U23: LATCH SOLENOID DRIVER + CLAMP - TBD, symbol Module_U23
- added U24: ESP32 FEEDBACK / LATCH GPIO ASSIGNMENTS TBD, symbol Module_U24
- added Y1: ELECTRONIC LATCH - COIL VOLTAGE TBD, symbol Module_Y1
Connections:
- net MOTOR24: now also F23.1 (IN)
- net MOTOR_GND: now also J23.3 (GND), J24.4 (GND), U23.2 (GND)
- new net BUCKET_LOWERED: J24.1 (BUCKET_LOWERED), U24.4 (BUCKET_LOWERED)
- new net DOOR_CLOSED: J23.1 (DOOR_CLOSED), U24.2 (CLOSED_INPUT)
- new net EXCAVATOR_DEPLOYED: J24.3 (EXCAVATOR_DEPLOYED), U24.6 (EXCAVATOR_DEPLOYED)
- new net EXCAVATOR_STOWED: J24.2 (EXCAVATOR_STOWED), U24.5 (EXCAVATOR_STOWED)
- new net LATCH_24: F23.2 (OUT), U23.1 (VIN), Y1.1 (PLUS)
- new net LATCH_ENGAGED: J23.2 (LATCH_ENGAGED), U24.3 (ENGAGED_INPUT)
- new net LATCH_RELEASE: U23.3 (RELEASE_3V3), U24.1 (RELEASE)
- new net LATCH_SW: U23.4 (OUT), Y1.2 (SW_RETURN)
Other:
- title: Lunar Hawks Rev C - System Wiring Draft -> Lunar Hawks Rev C.1 - Top Hinged Door and Four Actuators

Commit message: Fix KiCad ERC grid, symbol library and sensor interface errors
Parts:
- removed BT1: 24V MOTOR BATTERY, symbol Module_BT1
- removed BT2: V-MOUNT COMPUTE BATTERY, symbol Module_BT2
- removed F1: MAIN FUSE - SIZE TBD, symbol Module_F1
- removed F10: FL BRANCH FUSE - TBD, symbol Module_F10
- removed F11: FR BRANCH FUSE - TBD, symbol Module_F11
- removed F12: RL BRANCH FUSE - TBD, symbol Module_F12
- removed F13: RR BRANCH FUSE - TBD, symbol Module_F13
- removed F2: COMPUTE FUSE - SIZE TBD, symbol Module_F2
- removed F20: CONVEYOR FUSE - TBD, symbol Module_F20
- removed F21: BUCKET FUSE - TBD, symbol Module_F21
- removed F22: LIFT FUSE - TBD, symbol Module_F22
- removed F23: LATCH BRANCH FUSE - TBD, symbol Module_F23
- removed F3: LOGIC FUSE - SIZE TBD, symbol Module_F3
- removed J20: CONVEYOR MOTOR, symbol Module_J20
- removed J21: BUCKET ACTUATOR PAIR; SYNC REQUIRED, symbol Module_J21
- removed J22: LIFT ACTUATOR PAIR; SYNC REQUIRED, symbol Module_J22
- removed J23: DOOR / LATCH FEEDBACK INTERFACE, symbol Module_J23
- removed J24: ACTUATOR ENDPOINT FEEDBACK, symbol Module_J24
- removed K1: DC CONTACTOR - RATING TBD, symbol Module_K1
- removed M1: FL BLDC MOTOR, symbol Module_M1
- removed M2: FR BLDC MOTOR, symbol Module_M2
- removed M3: RL BLDC MOTOR, symbol Module_M3
- removed M4: RR BLDC MOTOR, symbol Module_M4
- removed SW1: LATCHING E-STOP NC, symbol Module_SW1
- removed U1: CARRIER INPUT PROTECTION / DC-DC, symbol Module_U1
- removed U10: FL EXTERNAL BLDC CONTROLLER, symbol Module_U10
- removed U11: FR EXTERNAL BLDC CONTROLLER, symbol Module_U11
- removed U12: RL EXTERNAL BLDC CONTROLLER, symbol Module_U12
- removed U13: RR EXTERNAL BLDC CONTROLLER, symbol Module_U13
- removed U2: JETSON ORIN NX CARRIER - MODEL TBD, symbol Module_U2
- removed U20: CONVEYOR EXTERNAL BRUSHED DRIVER, symbol Module_U20
- removed U21: BUCKET EXTERNAL BRUSHED DRIVER, symbol Module_U21
- removed U22: LIFT EXTERNAL BRUSHED DRIVER, symbol Module_U22
- removed U23: LATCH SOLENOID DRIVER + CLAMP - TBD, symbol Module_U23
- removed U24: ESP32 FEEDBACK / LATCH GPIO ASSIGNMENTS TBD, symbol Module_U24
- removed U3: ISOLATED UART MODULE 115200, symbol Module_U3
- removed U4: COMPUTE 3V3 REGULATOR MODULE, symbol Module_U4
- removed U5: 24V TO 3V3 REGULATOR MODULE, symbol Module_U5
- removed U6: ESP32 WROOM INTERFACE - GPIO TBD, symbol Module_U6
- removed Y1: ELECTRONIC LATCH - COIL VOLTAGE TBD, symbol Module_Y1
- added BT1: 24V MOTOR BATTERY, symbol LunarHawks:Module_BT1
- added BT2: V-MOUNT COMPUTE BATTERY, symbol LunarHawks:Module_BT2
- added F1: MAIN FUSE - SIZE TBD, symbol LunarHawks:Module_F1
- added F10: FL BRANCH FUSE - TBD, symbol LunarHawks:Module_F10
- added F11: FR BRANCH FUSE - TBD, symbol LunarHawks:Module_F11
- added F12: RL BRANCH FUSE - TBD, symbol LunarHawks:Module_F12
- added F13: RR BRANCH FUSE - TBD, symbol LunarHawks:Module_F13
- added F2: COMPUTE FUSE - SIZE TBD, symbol LunarHawks:Module_F2
- added F20: CONVEYOR FUSE - TBD, symbol LunarHawks:Module_F20
- added F21: BUCKET FUSE - TBD, symbol LunarHawks:Module_F21
- added F22: LIFT FUSE - TBD, symbol LunarHawks:Module_F22
- added F23: LATCH BRANCH FUSE - TBD, symbol LunarHawks:Module_F23
- added F3: LOGIC FUSE - SIZE TBD, symbol LunarHawks:Module_F3
- added J20: CONVEYOR MOTOR, symbol LunarHawks:Module_J20
- added J21: BUCKET ACTUATOR PAIR; SYNC REQUIRED, symbol LunarHawks:Module_J21
- added J22: LIFT ACTUATOR PAIR; SYNC REQUIRED, symbol LunarHawks:Module_J22
- added J23: DOOR / LATCH FEEDBACK INTERFACE, symbol LunarHawks:Module_J23
- added J24: ACTUATOR ENDPOINT FEEDBACK, symbol LunarHawks:Module_J24
- added J25: LIDAR USB INTERFACE, symbol LunarHawks:Module_J25
- added J26: CAMERA USB INTERFACE, symbol LunarHawks:Module_J26
- added K1: DC CONTACTOR - RATING TBD, symbol LunarHawks:Module_K1
- added M1: FL BLDC MOTOR, symbol LunarHawks:Module_M1
- added M2: FR BLDC MOTOR, symbol LunarHawks:Module_M2
- added M3: RL BLDC MOTOR, symbol LunarHawks:Module_M3
- added M4: RR BLDC MOTOR, symbol LunarHawks:Module_M4
- added SW1: LATCHING E-STOP NC, symbol LunarHawks:Module_SW1
- added U1: CARRIER INPUT PROTECTION / DC-DC, symbol LunarHawks:Module_U1
- added U10: FL EXTERNAL BLDC CONTROLLER, symbol LunarHawks:Module_U10
- added U11: FR EXTERNAL BLDC CONTROLLER, symbol LunarHawks:Module_U11
- added U12: RL EXTERNAL BLDC CONTROLLER, symbol LunarHawks:Module_U12
- added U13: RR EXTERNAL BLDC CONTROLLER, symbol LunarHawks:Module_U13
- added U2: JETSON ORIN NX CARRIER - MODEL TBD, symbol LunarHawks:Module_U2
- added U20: CONVEYOR EXTERNAL BRUSHED DRIVER, symbol LunarHawks:Module_U20
- added U21: BUCKET EXTERNAL BRUSHED DRIVER, symbol LunarHawks:Module_U21
- added U22: LIFT EXTERNAL BRUSHED DRIVER, symbol LunarHawks:Module_U22
- added U23: LATCH SOLENOID DRIVER + CLAMP - TBD, symbol LunarHawks:Module_U23
- added U24: ESP32 FEEDBACK / LATCH GPIO ASSIGNMENTS TBD, symbol LunarHawks:Module_U24
- added U3: ISOLATED UART MODULE 115200, symbol LunarHawks:Module_U3
- added U4: COMPUTE 3V3 REGULATOR MODULE, symbol LunarHawks:Module_U4
- added U5: 24V TO 3V3 REGULATOR MODULE, symbol LunarHawks:Module_U5
- added U6: ESP32 WROOM INTERFACE - GPIO TBD, symbol LunarHawks:Module_U6
- added Y1: ELECTRONIC LATCH - COIL VOLTAGE TBD, symbol LunarHawks:Module_Y1
Connections:
- net BAT24_FUSED: now also F1.2 (OUT), F3.1 (IN), K1.1 (POWER_IN), SW1.1 (IN)
- net BAT24_RAW: now also BT1.1 (PLUS), F1.1 (IN)
- net BUCKET_24: now also F21.2 (OUT), U21.1 (VIN)
- net BUCKET_A: now also J21.1 (A), U21.5 (OUT_A)
- net BUCKET_B: now also J21.2 (B), U21.6 (OUT_B)
- net BUCKET_DOWN: now also U21.4 (BUCKET_DOWN), U6.11 (BUCKET_DOWN)
- net BUCKET_LOWERED: now also J24.1 (BUCKET_LOWERED), U24.4 (BUCKET_LOWERED)
- net BUCKET_UP: now also U21.3 (BUCKET_UP), U6.10 (BUCKET_UP)
- net COMPUTE_3V3: now also U3.1 (A_VCC), U4.3 (OUT)
- net COMPUTE_FUSED: now also F2.2 (OUT), U1.1 (IN_PLUS)
- net COMPUTE_GND: now also BT2.2 (MINUS), U1.2 (IN_RETURN), U1.4 (OUT_RETURN), U2.2 (GND), U3.2 (A_GND), U4.2 (RETURN)
- net COMPUTE_RAW: now also BT2.1 (PLUS), F2.1 (IN)
- net CONVEYOR_24: now also F20.2 (OUT), U20.1 (VIN)
- net CONVEYOR_A: now also J20.1 (A), U20.4 (OUT_A)
- net CONVEYOR_B: now also J20.2 (B), U20.5 (OUT_B)
- net CONVEYOR_PWM: now also U20.3 (CONVEYOR_PWM), U6.9 (CONVEYOR)
- net DOOR_CLOSED: now also J23.1 (DOOR_CLOSED), U24.2 (CLOSED_INPUT)
- net ESP32_RX: now also U3.7 (B_RX), U6.3 (RX)
- net ESP32_TX: now also U3.8 (B_TX), U6.4 (TX)
- net ESTOP_COIL: now also K1.3 (COIL_PLUS), SW1.2 (OUT)
- net EXCAVATOR_DEPLOYED: now also J24.3 (EXCAVATOR_DEPLOYED), U24.6 (EXCAVATOR_DEPLOYED)
- net EXCAVATOR_STOWED: now also J24.2 (EXCAVATOR_STOWED), U24.5 (EXCAVATOR_STOWED)
- net FL_24: now also F10.2 (OUT), U10.1 (VIN)
- net FL_U: now also M1.1 (U), U10.5 (PHASE_U)
- net FL_V: now also M1.2 (V), U10.6 (PHASE_V)
- net FL_W: now also M1.3 (W), U10.7 (PHASE_W)
- net FR_24: now also F11.2 (OUT), U11.1 (VIN)
- net FR_U: now also M2.1 (U), U11.5 (PHASE_U)
- net FR_V: now also M2.2 (V), U11.6 (PHASE_V)
- net FR_W: now also M2.3 (W), U11.7 (PHASE_W)
- net JETSON_INPUT: now also U1.3 (OUT_PLUS), U2.1 (VIN), U4.1 (IN)
- net JETSON_RX: now also U2.4 (UART_RX_3V3), U3.4 (A_RX)
- net JETSON_TX: now also U2.3 (UART_TX_3V3), U3.3 (A_TX)
- net LATCH_24: now also F23.2 (OUT), U23.1 (VIN), Y1.1 (PLUS)
- net LATCH_ENGAGED: now also J23.2 (LATCH_ENGAGED), U24.3 (ENGAGED_INPUT)
- net LATCH_RELEASE: now also U23.3 (RELEASE_3V3), U24.1 (RELEASE)
- net LATCH_SW: now also U23.4 (OUT), Y1.2 (SW_RETURN)
- net LEFT_DIR: now also U10.4 (DIR), U12.4 (DIR), U6.6 (LEFT_DIR)
- net LEFT_PWM: now also U10.3 (PWM), U12.3 (PWM), U6.5 (LEFT_PWM)
- net LIFT_24: now also F22.2 (OUT), U22.1 (VIN)
- net LIFT_A: now also J22.1 (A), U22.5 (OUT_A)
- net LIFT_B: now also J22.2 (B), U22.6 (OUT_B)
- net LIFT_DOWN: now also U22.4 (LIFT_DOWN), U6.13 (LIFT_DOWN)
- net LIFT_UP: now also U22.3 (LIFT_UP), U6.12 (LIFT_UP)
- net LOGIC_3V3: now also U3.5 (B_VCC), U5.3 (VOUT), U6.1 (VCC)
- net LOGIC_INPUT: now also F3.2 (OUT), U5.1 (VIN)
- net MOTOR24: now also F10.1 (IN), F11.1 (IN), F12.1 (IN), F13.1 (IN), F20.1 (IN), F21.1 (IN), F22.1 (IN), F23.1 (IN), K1.2 (POWER_OUT)
- net MOTOR_GND: now also BT1.2 (MINUS), J23.3 (GND), J24.4 (GND), K1.4 (COIL_MINUS), U10.2 (GND), U11.2 (GND), U12.2 (GND), U13.2 (GND), U20.2 (GND), U21.2 (GND), U22.2 (GND), U23.2 (GND), U3.6 (B_GND), U5.2 (GND), U6.2 (GND)
- net RIGHT_DIR: now also U11.4 (DIR), U13.4 (DIR), U6.8 (RIGHT_DIR)
- net RIGHT_PWM: now also U11.3 (PWM), U13.3 (PWM), U6.7 (RIGHT_PWM)
- net RL_24: now also F12.2 (OUT), U12.1 (VIN)
- net RL_U: now also M3.1 (U), U12.5 (PHASE_U)
- net RL_V: now also M3.2 (V), U12.6 (PHASE_V)
- net RL_W: now also M3.3 (W), U12.7 (PHASE_W)
- net RR_24: now also F13.2 (OUT), U13.1 (VIN)
- net RR_U: now also M4.1 (U), U13.5 (PHASE_U)
- net RR_V: now also M4.2 (V), U13.6 (PHASE_V)
- net RR_W: now also M4.3 (W), U13.7 (PHASE_W)
- net USB_CAMERA: now also J26.1 (USB), U2.6 (USB_CAMERA)
- net USB_LIDAR: now also J25.1 (USB), U2.5 (USB_LIDAR)
