Commit message: Reinforce wheel and resize to 248 mm for 256 mm print bed

File: ros2_ws/src/lunabotics_description/urdf/lunar_hawks.urdf (robot description, URDF)
Before this commit: robot lunar_hawks, 33 links, 32 joints
Links:
- link wheel_fl: geometry collision cylinder length=0.1 radius=0.124; visual mesh filename=package://lunabotics_description/meshes/wheel.stl scale=.001 .001 .001
- link wheel_fr: geometry collision cylinder length=0.1 radius=0.124; visual mesh filename=package://lunabotics_description/meshes/wheel.stl scale=.001 .001 .001
- link wheel_rl: geometry collision cylinder length=0.1 radius=0.124; visual mesh filename=package://lunabotics_description/meshes/wheel.stl scale=.001 .001 .001
- link wheel_rr: geometry collision cylinder length=0.1 radius=0.124; visual mesh filename=package://lunabotics_description/meshes/wheel.stl scale=.001 .001 .001

Commit message: Add swept thin-tip grousers and removable wheel cavity covers

File: ros2_ws/src/lunabotics_description/urdf/lunar_hawks.urdf (robot description, URDF)
Before this commit: robot lunar_hawks, 33 links, 32 joints
Links:
- link wheel_fl: geometry collision cylinder length=0.1 radius=0.124; visual mesh filename=package://lunabotics_description/meshes/wheel_assembled.stl scale=.001 .001 .001
- link wheel_fr: geometry collision cylinder length=0.1 radius=0.124; visual mesh filename=package://lunabotics_description/meshes/wheel_assembled.stl scale=.001 .001 .001
- link wheel_rl: geometry collision cylinder length=0.1 radius=0.124; visual mesh filename=package://lunabotics_description/meshes/wheel_assembled.stl scale=.001 .001 .001
- link wheel_rr: geometry collision cylinder length=0.1 radius=0.124; visual mesh filename=package://lunabotics_description/meshes/wheel_assembled.stl scale=.001 .001 .001

Commit message: Gate mission startup on stable simulation clock and clear camera from LiDAR plane

File: ros2_ws/src/lunabotics_description/urdf/lunar_hawks.urdf (robot description, URDF)
Before this commit: robot lunar_hawks, 33 links, 32 joints
Joints:
- joint camera_mount: origin xyz=.36 0 .48 rpy=0 0 0 -> xyz=.36 0 .42 rpy=0 0 0

Commit message: Prevent simulated LiDAR self-returns

File: ros2_ws/src/lunabotics_description/urdf/lunar_hawks.urdf (robot description, URDF)
Before this commit: robot lunar_hawks, 33 links, 32 joints
Links:
- link camera_link: geometry visual box size=.04 .04 .04
- link lidar_link: geometry visual box size=.04 .04 .04
Joints:
- joint lidar_mount: origin xyz=.15 0 .5 rpy=0 0 0 -> xyz=.15 0 .62 rpy=0 0 0

Commit message: Place simulated LiDAR above rover self-occlusion

File: ros2_ws/src/lunabotics_description/urdf/lunar_hawks.urdf (robot description, URDF)
Before this commit: robot lunar_hawks, 33 links, 32 joints
Joints:
- joint lidar_mount: origin xyz=.15 0 .62 rpy=0 0 0 -> xyz=0 0 .85 rpy=0 0 0
